File: kazhan.kicad_pcb (KiCad board)
At the start: 2 copper layers, 91 parts, among them J1 USB_C_Receptacle_USB2.0, J2 USB_C_Receptacle_USB2.0, J3 USB_C_Receptacle_USB2.0, SW3 BOOT, SW4 RESET, U1 USBLC6-2SC6, U2 CH552T, U3 CH552T, U4 USBLC6-2SC6, U5 CH552T

Commit message: outline and placing started
Parts:
- added H1: Mounting_Hole, MyFootprintsCollection:MountingHole_3.5mmX4.5mm_Pad, F.Cu at (37.2, 77.1)
- added H2: Mounting_Hole, MyFootprintsCollection:MountingHole_3.5mmX4.5mm_Pad, F.Cu at (130.5, 46.0)
- added H3: Mounting_Hole, MyFootprintsCollection:MountingHole_3.5mmX4.5mm_Pad, F.Cu at (77.0, 32.7)
- added H4: Mounting_Hole, MyFootprintsCollection:MountingHole_3.5mmX4.5mm_Pad, F.Cu at (105.3, 109.0)
- added H5: Mounting_Hole, MyFootprintsCollection:MountingHole_3.5mmX4.5mm_Pad, F.Cu at (155.9, 144.8)
- D1, D12, D13, D16, D3, D5, D7, D9, SW1, U2: moved to B.Cu
- J1: value USB_C_Receptacle_USB2.0 -> AudioJack4; footprint Connector_USB:USB_C_Receptacle_HRO_TYPE-C-31-M-12 -> MyFootprintsCollection:PJ-320A-REVERSIBLE-F.Cu-placing
- J2: value USB_C_Receptacle_USB2.0 -> AudioJack4; footprint Connector_USB:USB_C_Receptacle_HRO_TYPE-C-31-M-12 -> MyFootprintsCollection:PJ-320A-REVERSIBLE-B.Cu-placing
- JP10, JP14, JP18, JP6: footprint Jumper:SolderJumper-2_P1.3mm_Open_RoundedPad1.0x1.5mm -> MyFootprintsCollection:SolderJumper-EdgeCut-B.Cu-Placing
- JP13, JP17, JP5, JP9: footprint Jumper:SolderJumper-2_P1.3mm_Open_RoundedPad1.0x1.5mm -> MyFootprintsCollection:SolderJumper-EdgeCut-F.Cu-Placing
- JP23: footprint Jumper:SolderJumper-2_P1.3mm_Open_RoundedPad1.0x1.5mm -> MyFootprintsCollection:SolderJumper-F.Cu-B.Cu
- S1, S10, S11, S12, S17, S18, S19, S2, S23, S24, S25, S3, S4, S9: footprint MyFootprintsCollection:SW_Hotswap_Kailh_Choc_MX_1.00u -> MyFootprintsCollection:SW_Hotswap_Kailh_Choc_MX_1.00u_One_Sided
- S13, S14, S15, S16, S20, S21, S22, S26, S27, S28, S5, S6, S7, S8: footprint MyFootprintsCollection:SW_Hotswap_Kailh_Choc_MX_1.00u -> MyFootprintsCollection:SW_Hotswap_Kailh_Choc_MX_1.00u_One_Sided; moved to B.Cu
- U5: footprint Package_SO:TSSOP-20_4.4x6.5mm_P0.65mm -> MyFootprintsCollection:TSSOP-20_4.4x6.5mm_P0.65mm-REVERSIBLE
- moved S28 219.7 mm to (57.6, 69.3), turned to 163 degrees
- moved S7 219.3 mm to (114.9, 46.5), turned to 153 degrees
- moved R2 213.8 mm to (156.0, 57.8), turned to 90 degrees
- moved R3 210.3 mm to (156.0, 63.4), turned to -90 degrees
- moved D18 204.5 mm to (158.7, 67.2), turned to -90 degrees
- moved SW4 201.3 mm to (148.2, 65.5), turned to -117 degrees
- moved C1 200.9 mm to (156.2, 67.2), turned to 90 degrees
- moved R4 200.7 mm to (161.5, 67.1), turned to 90 degrees
- moved R1 200.3 mm to (151.4, 70.0), turned to 153 degrees
- moved SW3 198.8 mm to (142.8, 62.6), turned to 63 degrees
- moved F1 198.3 mm to (166.6, 68.5), turned to 180 degrees
- moved C2 197.5 mm to (161.7, 72.0), turned to 90 degrees
- moved R5 197.3 mm to (166.8, 71.9), turned to 90 degrees
- moved D19 195.9 mm to (166.1, 77.0)
- moved U4 192.8 mm to (158.0, 71.6)
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Connections:
- net RX renamed L_RX
- net TX renamed L_TX
- U1 pad 4: P_TX -> Net-(J1-PadR2)
- U1 pad 6: P_RX -> Net-(J1-PadR1)
- U2 pad 10: Net-(U2-P30) -> R_RX
- U2 pad 9: Net-(U2-P31) -> R_TX
Other:
- board outline added: 143.6 x 139.6 mm
- board text added: "-17"
- board text added: "-22"
- board text added: "-27"
- board text added: "-41,998"
- board text added: "-70"
