File: kazhan_oldCopy.kicad_pcb (KiCad board)
At the start: 2 copper layers, 143.6 x 139.6 mm, 99 parts, among them J1 AudioJack4, J2 AudioJack4, J3 USB_C_Receptacle_USB2.0, SW3 BOOT, SW4 RESET, SW5 BOOT, SW6 RESET, U1 USBLC6-2SC6, U2 CH552T, U3 CH552T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

Commit message: all except matrix is routed
Parts:
- removed JP1: SolderJumper_2_Open, MyFootprintsCollection:SolderJumper-F.Cu-B.Cu
- moved SW5 103.9 mm to (212.2, 72.4), turned to 180 degrees
- moved R6 87.9 mm to (206.1, 70.3), turned to 180 degrees
- moved SW6 78.8 mm to (212.2, 78.5), turned to 180 degrees
- moved R1 41.2 mm to (151.4, 70.0)
- moved SW3 39.9 mm to (142.8, 62.6), turned to 63 degrees
- moved U2 29.1 mm to (152.5, 97.5)
- moved JP20 27.6 mm to (160.3, 104.1), turned to 0 degrees
- moved JP19 27.5 mm to (160.3, 104.1), turned to 180 degrees
- moved JP21 26.2 mm to (160.2, 102.8), turned to 180 degrees
- moved JP22 26.1 mm to (160.2, 102.8), turned to 0 degrees
- moved U1 22.7 mm to (152.0, 87.8), turned to 0 degrees
- moved J2 19.5 mm to (168.8, 80.8)
- moved J1 19.5 mm to (168.8, 80.7)
- moved F1 19.0 mm to (166.1, 67.0), turned to 180 degrees
- moved J3 18.6 mm to (163.1, 60.0), turned to 180 degrees
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Connections:
- SW5 pad 2: Net-(SW5-B) -> +3.3V
- SW6 pad 2: Net-(SW5-B) -> +3.3V
- U2 pad 20: Net-(SW5-B) -> +3.3V
Routing:
- net Net-(SW5-B): track 63.6 -> 0.00 mm
- net Net-(U2-P36): track 56.5 -> 0.00 mm, vias 2 -> 0
- net VCC: track 91.6 -> 41.3 mm, vias 4 -> 1
- net ROW2: track 41.4 -> 0.00 mm, vias 2 -> 0
- net ROW4: track 30.7 -> 0.00 mm, vias 4 -> 0
- net COL3: track 31.3 -> 6.32 mm
- net ROW3: track 22.1 -> 0.00 mm, vias 2 -> 0
- net L_RX: track 20.3 -> 0.00 mm, vias 2 -> 0
- net L_TX: track 17.9 -> 0.00 mm, vias 2 -> 0
- net RST: track 72.7 -> 56.2 mm, vias 4 -> 0
- net COL1: track 0.00 -> 15.8 mm
- net Net-(D15-A-Pad2): track 0.00 -> 14.8 mm
- net R_COL2: track 14.1 -> 0.00 mm
- net R_COL1: track 14.1 -> 0.00 mm, vias 2 -> 0
- net Net-(D10-K): track 13.1 -> 0.00 mm, vias 2 -> 0
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- added copper zone on B.Cu, net GND
- added copper zone on F.Cu, net GND
